Commit message: not working lidar , but the latest version

File: install/four_diff_drive_description/share/four_diff_drive_description/urdf/four_diff_drive.xacro (robot description, xacro)
@@ -1 +1,174 @@
-/home/orinnano256/Desktop/IAST_stuff_2_test_lidar/build/four_diff_drive_description/urdf/four_diff_drive.xacro
+<?xml version="1.0" ?>
+<robot name="four_diff_drive" xmlns:xacro="http://www.ros.org/wiki/xacro">
+<xacro:include filename="$(find four_diff_drive_description)/urdf/materials.xacro" />
+<xacro:include filename="$(find four_diff_drive_description)/urdf/four_diff_drive.trans" />
+<xacro:include filename="$(find four_diff_drive_description)/urdf/four_diff_drive.gazebo" />
+<link name="world_link"/>
+<link name="base_link">
+  <inertial>
+    <origin xyz="0.38933319773372493 0.025457111892628326 0.14121510359167855" rpy="0 0 0"/>
+    <mass value="109.04860734197118"/>
+    <inertia ixx="13.295168" iyy="14.356455" izz="2.822404" ixy="-0.010501" iyz="0.671179" ixz="0.044683"/>
+  </inertial>
+  <visual>
+    <origin xyz="0 0 0" rpy="0 0 0"/>
+    <geometry>
+      <mesh filename="file://$(find four_diff_drive_description)/meshes/base_link.stl" scale="0.001 0.001 0.001"/>
+    </geometry>
+    <material name="silver"/>
+  </visual>
+  <collision>
+    <origin xyz="0 0 0" rpy="0 0 0"/>
+    <geometry>
+      <mesh filename="file://$(find four_diff_drive_description)/meshes/base_link.stl" scale="0.001 0.001 0.001"/>
+    </geometry>
+  </collision>
+</link>
+<link name="fr_wheel_1_1">
+  <inertial>
+    <origin xyz="-0.0006678192662164517 7.879899210916363e-08 -5.297525051961571e-08" rpy="0 0 0"/>
+    <mass value="13.66073272140364"/>
+    <inertia ixx="0.11786" iyy="0.062234" izz="0.062234" ixy="-0.0" iyz="0.0" ixz="0.0"/>
+  </inertial>
+  <visual>
+    <origin xyz="-0.177234 0.134788 -0.628175" rpy="0 0 0"/>
+    <geometry>
+      <mesh filename="file://$(find four_diff_drive_description)/meshes/fr_wheel_1_1.stl" scale="0.001 0.001 0.001"/>
+    </geometry>
+    <material name="silver"/>
+  </visual>
+  <collision>
+    <origin xyz="-0.177234 0.134788 -0.628175" rpy="0 0 0"/>
+    <geometry>
+      <mesh filename="file://$(find four_diff_drive_description)/meshes/fr_wheel_1_1.stl" scale="0.001 0.001 0.001"/>
+    </geometry>
+  </collision>
+</link>
+<link name="fl_wheel_1_1">
+  <inertial>
+    <origin xyz="0.0006669561985305217 1.5491755467333945e-07 -1.2909381374992535e-07" rpy="0 0 0"/>
+    <mass value="13.660732721403573"/>
+    <inertia ixx="0.11786" iyy="0.062234" izz="0.062234" ixy="-0.0" iyz="0.0" ixz="0.0"/>
+  </inertial>
+  <visual>
+    <origin xyz="-0.599734 0.134788 -0.628175" rpy="0 0 0"/>
+    <geometry>
+      <mesh filename="file://$(find four_diff_drive_description)/meshes/fl_wheel_1_1.stl" scale="0.001 0.001 0.001"/>
+    </geometry>
+    <material name="silver"/>
+  </visual>
+  <collision>
+    <origin xyz="-0.599734 0.134788 -0.628175" rpy="0 0 0"/>
+    <geometry>
+      <mesh filename="file://$(find four_diff_drive_description)/meshes/fl_wheel_1_1.stl" scale="0.001 0.001 0.001"/>
+    </geometry>
+  </collision>
+</link>
+<link name="rr_wheel_1_1">
+  <inertial>
+    <origin xyz="-0.0006678192662164517 1.9850436036583652e-07 -1.2911571540402678e-07" rpy="0 0 0"/>
+    <mass value="13.660732721403626"/>
+    <inertia ixx="0.11786" iyy="0.062234" izz="0.062234" ixy="-0.0" iyz="-0.0" ixz="-0.0"/>
+  </inertial>
+  <visual>
+    <origin xyz="-0.177234 0.134788 0.038075" rpy="0 0 0"/>
+    <geometry>
+      <mesh filename="file://$(find four_diff_drive_description)/meshes/rr_wheel_1_1.stl" scale="0.001 0.001 0.001"/>
+    </geometry>
+    <material name="silver"/>
+  </visual>
+  <collision>
+    <origin xyz="-0.177234 0.134788 0.038075" rpy="0 0 0"/>
+    <geometry>
+      <mesh filename="file://$(find four_diff_drive_description)/meshes/rr_wheel_1_1.stl" scale="0.001 0.001 0.001"/>
+    </geometry>
+  </collision>
+</link>
+<link name="rl_wheel_1_1">
+  <inertial>
+    <origin xyz="0.0006669561985307437 1.5491755470109503e-07 -1.291157157232159e-07" rpy="0 0 0"/>
+    <mass value="13.660732721403523"/>
+    <inertia ixx="0.11786" iyy="0.062234" izz="0.062234" ixy="-0.0" iyz="0.0" ixz="0.0"/>
+  </inertial>
+  <visual>
+    <origin xyz="-0.599734 0.134788 0.038075" rpy="0 0 0"/>
+    <geometry>
+      <mesh filename="file://$(find four_diff_drive_description)/meshes/rl_wheel_1_1.stl" scale="0.001 0.001 0.001"/>
+    </geometry>
+    <material name="silver"/>
+  </visual>
+  <collision>
+    <origin xyz="-0.599734 0.134788 0.038075" rpy="0 0 0"/>
+    <geometry>
+      <mesh filename="file://$(find four_diff_drive_description)/meshes/rl_wheel_1_1.stl" scale="0.001 0.001 0.001"/>
+    </geometry>
+  </collision>
+</link>
+<joint name="world_frame" type="fixed">
+  <origin xyz="0.0 0.0 0.0" rpy="1.57 0 0"/>
+  <parent link="world_link"/>
+  <child link="base_link"/>
+</joint>
+<joint name="fr_wheel_joint" type="continuous">
+  <origin xyz="0.177234 -0.134788 0.628175" rpy="0 0 0"/>
+  <parent link="base_link"/>
+  <child link="fr_wheel_1_1"/>
+  <axis xyz="1.0 0.0 0.0"/>
+</joint>
+<joint name="fl_wheel_joint" type="continuous">
+  <origin xyz="0.599734 -0.134788 0.628175" rpy="0 0 0"/>
+  <parent link="base_link"/>
+  <child link="fl_wheel_1_1"/>
+  <axis xyz="1.0 0.0 0.0"/>
+</joint>
+<joint name="rr_wheel_joint" type="continuous">
+  <origin xyz="0.177234 -0.134788 -0.038075" rpy="0 0 0"/>
+  <parent link="base_link"/>
+  <child link="rr_wheel_1_1"/>
+  <axis xyz="1.0 0.0 0.0"/>
+</joint>
+<joint name="rl_wheel_joint" type="continuous">
+  <origin xyz="0.599734 -0.134788 -0.038075" rpy="0 0 0"/>
+  <parent link="base_link"/>
+  <child link="rl_wheel_1_1"/>
+  <axis xyz="1.0 0.0 0.0"/>
+</joint>
+<ros2_control name="GazeboSimSystem" type="system">
+    <hardware>
+      <plugin>gazebo_ros2_control/GazeboSystem</plugin>
+    </hardware>
+    <joint name="fr_wheel_joint">
+      <command_interface name="velocity"/>
+      <state_interface name="position"/>
+      <state_interface name="velocity"/>
+    </joint>
+    <joint name="fl_wheel_joint">
+      <command_interface name="velocity"/>
+      <state_interface name="position"/>
+      <state_interface name="velocity"/>
+    </joint>
+    <joint name="rr_wheel_joint">
+      <command_interface name="velocity"/>
+      <state_interface name="position"/>
+      <state_interface name="velocity"/>
+    </joint>
+    <joint name="rl_wheel_joint">
+      <command_interface name="velocity"/>
+      <state_interface name="position"/>
+      <state_interface name="velocity"/>
+    </joint>
+</ros2_control>
+  <gazebo>
+    <plugin filename="libgazebo_ros2_control.so" name="gazebo_ros2_control">
+      <parameters>$(find four_diff_drive_description)/config/controller.yaml</parameters>
+    </plugin>
+    <plugin name="gazebo_ros_joint_state_publisher"
+        filename="libgazebo_ros_joint_state_publisher.so">
+        <update_rate>60</update_rate>
+        <joint_name>fr_wheel_joint</joint_name>
+        <joint_name>fl_wheel_joint</joint_name>
+        <joint_name>rr_wheel_joint</joint_name>
+        <joint_name>rl_wheel_joint</joint_name>
+    </plugin>
+  </gazebo>
+</robot>

File: install/four_diff_drive_description/share/four_diff_drive_description/urdf/materials.xacro (robot description, xacro)
@@ -1 +1,6 @@
-/home/orinnano256/Desktop/IAST_stuff_2_test_lidar/build/four_diff_drive_description/urdf/materials.xacro
+<?xml version="1.0" ?>
+<robot name="four_diff_drive" xmlns:xacro="http://www.ros.org/wiki/xacro" >
+<material name="silver">
+  <color rgba="0.700 0.700 0.700 1.000"/>
+</material>
+</robot>
