Commit message: The car is driving on the ground

File: install/four_diff_drive_description/share/four_diff_drive_description/urdf/four_diff_drive.urdf (robot description, URDF)
Before this commit: robot four_diff_drive, 7 links, 6 joints
Joints:
- joint odom_frame: origin xyz=0.0 0.0 0.0 rpy=0 0 0 -> xyz=0.599734 -0.134788 1.028175 rpy=0 0 0
- joint world_frame: origin xyz=0.0 0.0 0.0 rpy=1.57 0 0 -> xyz=0.0 0.0 0.245 rpy=0 0 0

Commit message: my RGB camera is added and displays the image

File: install/four_diff_drive_description/share/four_diff_drive_description/urdf/four_diff_drive.urdf (robot description, URDF)
Before this commit: robot four_diff_drive, 7 links, 6 joints
Links:
- added link camera_link; visual box size=0.010 0.03 0.03
- added link camera_link_optical
Joints:
- added joint camera_joint: type fixed, parent base_link, child camera_link, origin xyz=0.405 -0.05 0.98 rpy=0 -1.57 -1.57
- added joint camera_optical_joint: type fixed, parent camera_link, child camera_link_optical, origin xyz=0 0 0 rpy=-1.57 0 -1.57

Commit message: My lidar is added and it is scanning

File: install/four_diff_drive_description/share/four_diff_drive_description/urdf/four_diff_drive.urdf (robot description, URDF)
Before this commit: robot four_diff_drive, 9 links, 8 joints
Links:
- removed link camera_link
- removed link camera_link_optical
- added link laser_frame; collision box size=0.05 0.03 0.02; visual box size=0.05 0.03 0.02
- link base_link: geometry collision mesh filename=file:///home/orinnano/Desktop/IAST_stuff_2_test_lidar/insta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 scale=0.001 0.001 0.001; visual mesh filename=file:///home/orinnano/Desktop/IAST_stuff_2_test_lidar/insta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 scale=0.001 0.001 0.001
- link fl_wheel_1_1: geometry collision mesh filename=file:///home/orinnano/Desktop/IAST_stuff_2_test_lidar/insta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 scale=0.001 0.001 0.001; visual mesh filename=file:///home/orinnano/Desktop/IAST_stuff_2_test_lidar/insta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 scale=0.001 0.001 0.001
- link fr_wheel_1_1: geometry collision mesh filename=file:///home/orinnano/Desktop/IAST_stuff_2_test_lidar/insta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 scale=0.001 0.001 0.001; visual mesh filename=file:///home/orinnano/Desktop/IAST_stuff_2_test_lidar/insta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 scale=0.001 0.001 0.001
- link rl_wheel_1_1: geometry collision mesh filename=file:///home/orinnano/Desktop/IAST_stuff_2_test_lidar/insta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 scale=0.001 0.001 0.001; visual mesh filename=file:///home/orinnano/Desktop/IAST_stuff_2_test_lidar/insta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 scale=0.001 0.001 0.001
- link rr_wheel_1_1: geometry collision mesh filename=file:///home/orinnano/Desktop/IAST_stuff_2_test_lidar/insta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 scale=0.001 0.001 0.001; visual mesh filename=file:///home/orinnano/Desktop/IAST_stuff_2_test_lidar/insta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 scale=0.001 0.001 0.001
Joints:
- removed joint camera_joint
- removed joint camera_optical_joint
- added joint laser_joint: type fixed, parent base_link, child laser_frame, origin xyz=0.405 -0.05 0.88 rpy=1.57 0 0

Commit message: partial map making

File: install/four_diff_drive_description/share/four_diff_drive_description/urdf/four_diff_drive.urdf (robot description, URDF)
Before this commit: robot four_diff_drive, 8 links, 7 joints
Links:
- added link map
Joints:
- added joint map_frame: type fixed, parent map, child odom, origin xyz=0.0 0.0 0.0 rpy=0 0 0
- joint world_frame: child odom -> map; origin xyz=0.0 0.0 0.245 rpy=0 0 0 -> xyz=0.0 0.0 0.245 rpy=1.0 0 0

Commit message: navigation withour reaching the final goal as the map is moving with the goal :x

File: install/four_diff_drive_description/share/four_diff_drive_description/urdf/four_diff_drive.urdf (robot description, URDF)
Before this commit: robot four_diff_drive, 9 links, 8 joints
Links:
- removed link world_link
Joints:
- removed joint world_frame
- joint map_frame: child world_link -> odom
- joint odom_frame: origin xyz=0.599734 -0.134788 1.028175 rpy=0 0 0 -> xyz=0.0 0.0 0.0 rpy=0 0 0

File: install/four_diff_drive_description/share/four_diff_drive_description/urdf/four_diff_drive.xacro (robot description, xacro)
@@ -4,5 +4,6 @@
 <xacro:include filename="$(find four_diff_drive_description)/urdf/four_diff_drive.trans" />
 <xacro:include filename="$(find four_diff_drive_description)/urdf/four_diff_drive.gazebo" />
-<link name="world_link"/>
+<link name="map"/>
+<link name="odom"/>
 <link name="base_link">
   <inertial>
@@ -105,9 +106,32 @@
   </collision>
 </link>
-<joint name="world_frame" type="fixed">
-  <origin xyz="0.0 0.0 0.0" rpy="1.57 0 0"/>
-  <parent link="world_link"/>
-  <child link="base_link"/>
-</joint>
+<link name="laser_frame">
+     <visual>
+        <geometry>
+          <box size="0.05 0.03 0.02"/>
+        </geometry>
+        <material name="red"/>
+     </visual>
+     <collision>
+        <geometry>
+          <box size="0.05 0.03 0.02"/>
+        </geometry>
+     </collision>
+  </link>
+<joint name="map_frame" type="fixed">
+  <origin xyz="0.0 0.0 0.0" rpy="0 0 0"/>  <!--rpy: before(1.57,0,0) for world to base joint-->
+  <parent link="map"/>
+  <child link="odom"/>
+</joint>
+<joint name="odom_frame" type="fixed">    <!--fixed-->
+    <origin rpy="0 0 0" xyz="0.0 0.0 0.0"/>  <!-- z changed from 0.628175 to 1.028175, x: 0.599734 to 0.999734, y: -0.134788 to -0.434788 - anisha-->
+    <parent link="odom"/>
+    <child link="base_link"/>  <!--0.599734 -0.134788 1.028175-->
+  </joint>
+<joint name="laser_joint" type="fixed">
+    <origin rpy="1.57 0 0" xyz="0.405 -0.05 0.88"/>  <!-- z changed from 0.628175 to 1.028175, x: 0.599734 to 0.999734, y: -0.134788 to -0.434788 - anisha-->
+    <parent link="base_link"/>
+    <child link="laser_frame"/>
+  </joint>
 <joint name="fr_wheel_joint" type="continuous">
   <origin xyz="0.177234 -0.134788 0.628175" rpy="0 0 0"/>
@@ -134,7 +158,7 @@
   <axis xyz="1.0 0.0 0.0"/>
 </joint>
-<ros2_control name="GazeboSimSystem" type="system">
+<ros2_control name="IgnitionSystem" type="system">
     <hardware>
-      <plugin>gazebo_ros2_control/GazeboSystem</plugin>
+      <plugin>ign_ros2_control/IgnitionSystem</plugin>
     </hardware>
     <joint name="fr_wheel_joint">
@@ -159,16 +183,69 @@
     </joint>
 </ros2_control>
-  <gazebo>
-    <plugin filename="libgazebo_ros2_control.so" name="gazebo_ros2_control">
-      <parameters>$(find four_diff_drive_description)/config/controller.yaml</parameters>
+     <gazebo>
+<!-- Global odometer plugin -->
+    <plugin
+      filename="ignition-gazebo-odometry-publisher-system"
+      name="ignition::gazebo::systems::OdometryPublisher">
+      <odom_publish_frequency>50</odom_publish_frequency>
+      <odom_topic>/odom</odom_topic>
+      <odom_frame>odom</odom_frame>   <!--changed from odom to map-->
+      <robot_base_frame>base_link</robot_base_frame>
+      <tf_topic>/odom/tf</tf_topic>
     </plugin>
-    <plugin name="gazebo_ros_joint_state_publisher"
-        filename="libgazebo_ros_joint_state_publisher.so">
-        <update_rate>60</update_rate>
+    <!-- Diff drive controller plugin -->
+    <plugin filename="gz-sim-diff-drive-system" name="gz::sim::systems::DiffDrive">
+   <!-- wheels -->
+      <right_joint>fr_wheel_joint</right_joint>
+      <left_joint>fl_wheel_joint</left_joint>
+      <right_joint>rr_wheel_joint</right_joint>
+      <left_joint>rl_wheel_joint</left_joint>
+      <frame_id>odom</frame_id>   <!--changed from odom to map-->
+      <child_frame_id>base_link</child_frame_id>
+      <topic>/cmd_vel</topic>
+      <odom_topic>/odom</odom_topic>
+      </plugin>
+      <!--  -->
+      <!--<odom_publisher_frequency>30</odom_publisher_frequency> -->
+      <!-- <tf_topic>/tf</tf_topic>  -->  <!--commented out to test- anisha-->
+      <!-- Joint group velocity controller plugin -->
+      <plugin filename="ignition-gazebo-joint-group-velocity-controller-system"
+            name="joint_group_velocity_controller">
         <joint_name>fr_wheel_joint</joint_name>
         <joint_name>fl_wheel_joint</joint_name>
         <joint_name>rr_wheel_joint</joint_name>
         <joint_name>rl_wheel_joint</joint_name>
-    </plugin>
-  </gazebo>
+        <topic>/joint_group_velocity_controller/commands</topic>
+        <update_rate>30</update_rate>
+      </plugin>
+    </gazebo>
+    <!-- new code added for lidar gazebo reference sensor - anisha, 18/11/2024 -->
+    <gazebo reference="laser_frame">
+      <material>Gazebo/Red</material>
+      <sensor name="gpu_lidar" type="gpu_lidar">
+         <pose>0 0 0 0 0 0</pose>
+         <topic>scan</topic>
+         <ignition_frame_id>laser_frame</ignition_frame_id>
+         <visualize>true</visualize>
+         <update_rate>10</update_rate>
+         <ray>
+            <scan>
+              <horizontal>
+                <samples>360</samples>
+                <min_angle>-3.14</min_angle>
+                <max_angle>3.14</max_angle>
+              </horizontal>
+            </scan>
+            <range>
+              <min>0.2</min>
+              <max>20</max>
+            </range>
+         </ray>
+         <plugin name="gz::sim::systems::Sensors" filename="gz-sim-sensors-system">
+          <!-- <frame_name>laser_frame</frame_name>    -->
+          <!-- <output_type>sensor_msgs/msg/LaserScan</output_type> -->
+        </plugin>
+        <point_cloud_topic>/scan/points</point_cloud_topic>
+      </sensor>
+   </gazebo>
 </robot>
